File: PCB/PiicoDev-Distance-Sensor-VL53L1X.sch (KiCad schematic (older format))
At the start: 24 parts, among them J1 , J2 , J3 , J4 , J5 , U1 VL35L1x

Commit message: Update resistor values - all 10k
Parts:
- R1: value 1k -> 10k
- R3, R4: value 4k7 -> 10k
Changed lines of the file:
@@
 P 7600 3350
 F 0 "R3" H 7670 3396 50  0000 L CNN
-F 1 "4k7" H 7670 3305 50  0000 L CNN
+F 1 "10k" H 7670 3305 50  0000 L CNN
 F 2 "Resistor_SMD:R_0402_1005Metric" V 7530 3350 50  0001 C CNN
 F 3 "~" H 7600 3350 50  0001 C CNN
@@
 P 7000 3350
 F 0 "R4" H 7070 3396 50  0000 L CNN
-F 1 "4k7" H 7070 3305 50  0000 L CNN
+F 1 "10k" H 7070 3305 50  0000 L CNN
 F 2 "Resistor_SMD:R_0402_1005Metric" V 6930 3350 50  0001 C CNN
 F 3 "~" H 7000 3350 50  0001 C CNN
@@
 P 2200 3750
 F 0 "R1" H 2270 3796 50  0000 L CNN
-F 1 "1k" H 2270 3705 50  0000 L CNN
+F 1 "10k" H 2270 3705 50  0000 L CNN
 F 2 "Resistor_SMD:R_0402_1005Metric" V 2130 3750 50  0001 C CNN
 F 3 "~" H 2200 3750 50  0001 C CNN
